Commit message: updated dimensions to match real robot

File: description/robot_core.urdf.xacro (robot description, xacro)
@@ -32,5 +32,5 @@
     <parent link="base_link" />
     <child link="left_front_wheel" />
-    <origin xyz="0.22 0.3 -0.1" rpy="-${pi/2} 0 0" />
+    <origin xyz="0.2465 0.305 -0.0767" rpy="-${pi/2} 0 0" />
     <axis xyz="0 0 1" />
   </joint>
@@ -38,5 +38,5 @@
     <visual>
       <geometry>
-        <cylinder radius="0.15" length="0.14" />
+        <cylinder radius="0.19" length="0.14" />
       </geometry>
       <material name="gray" />
@@ -44,8 +44,8 @@
     <collision>
       <geometry>
-        <cylinder radius="0.15" length="0.14" />
+        <cylinder radius="0.19" length="0.14" />
       </geometry>
     </collision>
-        <xacro:inertial_cylinder mass="3" length="0.14" radius="0.15">
+        <xacro:inertial_cylinder mass="3" length="0.14" radius="0.19">
             <origin xyz="0 0 0" rpy="0 0 0"/>
         </xacro:inertial_cylinder>
@@ -54,5 +54,5 @@
     <parent link="base_link" />
     <child link="left_rear_wheel" />
-    <origin xyz="-0.22 0.3 -0.1" rpy="-${pi/2} 0 0" />
+    <origin xyz="-0.2465 0.305 -0.0767" rpy="-${pi/2} 0 0" />
     <axis xyz="0 0 1" />
   </joint>
@@ -60,5 +60,5 @@
     <visual>
       <geometry>
-        <cylinder radius="0.15" length="0.14" />
+        <cylinder radius="0.19" length="0.14" />
       </geometry>
       <material name="gray" />
@@ -66,8 +66,8 @@
     <collision>
       <geometry>
-        <cylinder radius="0.15" length="0.14" />
+        <cylinder radius="0.19" length="0.14" />
       </geometry>
     </collision>
-    <xacro:inertial_cylinder mass="3" length="0.14" radius="0.15">
+    <xacro:inertial_cylinder mass="3" length="0.14" radius="0.19">
       <origin xyz="0 0 0" rpy="0 0 0"/>
   </xacro:inertial_cylinder>
@@ -77,5 +77,5 @@
     <parent link="base_link" />
     <child link="right_front_wheel" />
-    <origin xyz="0.22 -0.3 -0.1" rpy="${pi/2} 0 0" />
+    <origin xyz="0.2465 -0.305 -0.0767" rpy="${pi/2} 0 0" />
     <axis xyz="0 0 -1" />
   </joint>
@@ -83,5 +83,5 @@
     <visual>
       <geometry>
-        <cylinder radius="0.15" length="0.14" />
+        <cylinder radius="0.19" length="0.14" />
       </geometry>
       <material name="gray" />
@@ -89,8 +89,8 @@
     <collision>
       <geometry>
-        <cylinder radius="0.15" length="0.14" />
+        <cylinder radius="0.19" length="0.14" />
       </geometry>
     </collision>
-    <xacro:inertial_cylinder mass="3" length="0.14" radius="0.15">
+    <xacro:inertial_cylinder mass="3" length="0.14" radius="0.19">
       <origin xyz="0 0 0" rpy="0 0 0"/>
   </xacro:inertial_cylinder>
@@ -99,5 +99,5 @@
     <parent link="base_link" />
     <child link="right_rear_wheel" />
-    <origin xyz="-0.22 -0.3 -0.1" rpy="${pi/2} 0 0" />
+    <origin xyz="-0.2465 -0.305 -0.0767" rpy="${pi/2} 0 0" />
     <axis xyz="0 0 -1" />
     <command_interface name="velocity" />
@@ -107,5 +107,5 @@
     <visual>
       <geometry>
-        <cylinder radius="0.15" length="0.14" />
+        <cylinder radius="0.19" length="0.14" />
       </geometry>
       <material name="gray" />
@@ -113,8 +113,8 @@
     <collision>
       <geometry>
-        <cylinder radius="0.15" length="0.14" />
+        <cylinder radius="0.19" length="0.14" />
       </geometry>
     </collision>
-    <xacro:inertial_cylinder mass="3" length="0.14" radius="0.15">
+    <xacro:inertial_cylinder mass="3" length="0.14" radius="0.19">
       <origin xyz="0 0 0" rpy="0 0 0"/>
   </xacro:inertial_cylinder>
