Commit message: added hardware configuration

File: description/robot.urdf.xacro (robot description, xacro)
@@ -1,233 +1,7 @@
 <?xml version="1.0"?>
-<robot xmlns:xacro="http://www.ros.org/wiki/xacro" name="robot">
-  <xacro:include filename="inertial_macros.xacro"/>
-  <material name="white">
-    <color rgba="1 1 1 1" />
-  </material>
-  <material name="blue">
-    <color rgba="0.2 0.2 1 1" />
-  </material>
-  <material name="gray">
-    <color rgba="0.3 0.3 0.3 1" />
-  </material>
-  <gazebo reference="frame">
-    <material>Gazebo/Blue</material>
-  </gazebo>
-  <gazebo reference="left_front_wheel">
-    <material>Gazebo/Gray</material>
-    <mu1 value='1' />
-    <mu2 value='1' />
-  </gazebo>
-  <gazebo reference="left_rear_wheel">
-    <material>Gazebo/Gray</material>
-    <mu1 value='1' />
-    <mu2 value='1' />
-  </gazebo>
-  <gazebo reference="right_front_wheel">
-    <material>Gazebo/Gray</material>
-    <mu1 value='1' />
-    <mu2 value='1' />
-  </gazebo>
-  <gazebo reference="right_rear_wheel">
-    <material>Gazebo/Gray</material>
-    <mu1 value='1' />
-    <mu2 value='1' />
-  </gazebo>
-  <!-- BASE LINK -->
-  <link name="base_link">
-  </link>
-  <!-- FRAME LINK -->
-  <joint name="frame_joint" type="fixed">
-    <parent link="base_link" />
-    <child link="frame" />
-    <origin xyz="0 0 0" />
-  </joint>
-  <link name="frame">
-    <visual>
-      <origin xyz="0 0 0" />
-      <geometry>
-        <box size="0.7 0.44 0.3" />
-      </geometry>
-      <material name="blue" />
-    </visual>
-    <collision>
-      <origin xyz="0 0 0" />
-      <geometry>
-        <box size="0.7 0.44 0.3" />
-      </geometry>
-    </collision>
-    <xacro:inertial_box mass="50" x="0.7" y="0.44" z="0.3">
-      <origin xyz="0 0 0" rpy="0 0 0"/>
-  </xacro:inertial_box>
-  </link>
-  <joint name="left_front_wheel_joint" type="continuous">
-    <mimic joint="left_rear_wheel_joint"/>
-    <parent link="base_link" />
-    <child link="left_front_wheel" />
-    <origin xyz="0.22 0.3 -0.1" rpy="-${pi/2} 0 0" />
-    <axis xyz="0 0 1" />
-  </joint>
-  <link name="left_front_wheel">
-    <visual>
-      <geometry>
-        <cylinder radius="0.15" length="0.14" />
-      </geometry>
-      <material name="gray" />
-    </visual>
-    <collision>
-      <geometry>
-        <cylinder radius="0.15" length="0.14" />
-      </geometry>
-    </collision>
-        <xacro:inertial_cylinder mass="3" length="0.14" radius="0.15">
-            <origin xyz="0 0 0" rpy="0 0 0"/>
-        </xacro:inertial_cylinder>
-  </link>
-  <joint name="left_rear_wheel_joint" type="continuous">
-    <parent link="base_link" />
-    <child link="left_rear_wheel" />
-    <origin xyz="-0.22 0.3 -0.1" rpy="-${pi/2} 0 0" />
-    <axis xyz="0 0 1" />
-  </joint>
-  <link name="left_rear_wheel">
-    <visual>
-      <geometry>
-        <cylinder radius="0.15" length="0.14" />
-      </geometry>
-      <material name="gray" />
-    </visual>
-    <collision>
-      <geometry>
-        <cylinder radius="0.15" length="0.14" />
-      </geometry>
-    </collision>
-    <xacro:inertial_cylinder mass="3" length="0.14" radius="0.15">
-      <origin xyz="0 0 0" rpy="0 0 0"/>
-  </xacro:inertial_cylinder>
-  </link>
-  <joint name="right_front_wheel_joint" type="continuous">
-    <mimic joint="right_rear_wheel_joint"/>
-    <parent link="base_link" />
-    <child link="right_front_wheel" />
-    <origin xyz="0.22 -0.3 -0.1" rpy="${pi/2} 0 0" />
-    <axis xyz="0 0 -1" />
-  </joint>
-  <link name="right_front_wheel">
-    <visual>
-      <geometry>
-        <cylinder radius="0.15" length="0.14" />
-      </geometry>
-      <material name="gray" />
-    </visual>
-    <collision>
-      <geometry>
-        <cylinder radius="0.15" length="0.14" />
-      </geometry>
-    </collision>
-    <xacro:inertial_cylinder mass="3" length="0.14" radius="0.15">
-      <origin xyz="0 0 0" rpy="0 0 0"/>
-  </xacro:inertial_cylinder>
-  </link>
-  <joint name="right_rear_wheel_joint" type="continuous">
-    <parent link="base_link" />
-    <child link="right_rear_wheel" />
-    <origin xyz="-0.22 -0.3 -0.1" rpy="${pi/2} 0 0" />
-    <axis xyz="0 0 -1" />
-    <command_interface name="velocity" />
-    <state_interface name="velocity" />
-  </joint>
-  <link name="right_rear_wheel">
-    <visual>
-      <geometry>
-        <cylinder radius="0.15" length="0.14" />
-      </geometry>
-      <material name="gray" />
-    </visual>
-    <collision>
-      <geometry>
-        <cylinder radius="0.15" length="0.14" />
-      </geometry>
-    </collision>
-    <xacro:inertial_cylinder mass="3" length="0.14" radius="0.15">
-      <origin xyz="0 0 0" rpy="0 0 0"/>
-  </xacro:inertial_cylinder>
-  </link>
-  <ros2_control name="GazeboSystem" type="system">
-    <hardware>
-      <plugin>gazebo_ros2_control/GazeboSystem</plugin>
-    </hardware>
-    <joint name="left_rear_wheel_joint">
-      <command_interface name="velocity">
-        <param name="min">-1</param>
-        <param name="max">1</param>
-      </command_interface>
-      <state_interface name="position" />
-      <state_interface name="velocity" />
-    </joint>
-    <joint name="right_rear_wheel_joint">
-      <command_interface name="velocity">
-        <param name="min">-1</param>
-        <param name="max">1</param>
-      </command_interface>
-      <state_interface name="position" />
-      <state_interface name="velocity" />
-    </joint>
-    <joint name="left_front_wheel_joint">
-      <param name="mimic">left_rear_wheel_joint</param>
-      <param name="multiplier">1</param>
-      <command_interface name="velocity">
-        <param name="min">-1</param>
-        <param name="max">1</param>
-      </command_interface>
-      <state_interface name="position" />
-      <state_interface name="velocity" />
-    </joint>
-    <joint name="right_front_wheel_joint">
-      <param name="mimic">right_rear_wheel_joint</param>
-      <param name="multiplier">1</param>
-      <command_interface name="velocity">
-        <param name="min">-1</param>
-        <param name="max">1</param>
-      </command_interface>
-      <state_interface name="position" />
-      <state_interface name="velocity" />
-    </joint>
-  </ros2_control>
-  <gazebo>
-    <plugin filename="libgazebo_ros2_control.so" name="gazebo_ros2_control">
-      <parameters>$(find outdoor_robot_one)/config/ros2_controllers.yaml</parameters>
-    </plugin>
-  </gazebo>
-  <gazebo reference="left_rear_wheel" >
-    <mu1>0.3</mu1>
-    <mu2>0.3</mu2>
-    <kp>1000000.0</kp>
-    <kd>100.0</kd>
-    <minDepth>0.0</minDepth>
-    <maxContacts>1</maxContacts>
-  </gazebo>
-  <gazebo reference="right_rear_wheel" >
-    <mu1>0.3</mu1>
-    <mu2>0.3</mu2>
-    <kp>1000000.0</kp>
-    <kd>100.0</kd>
-    <minDepth>0.0</minDepth>
-    <maxContacts>1</maxContacts>
-  </gazebo>
-  <gazebo reference="left_front_wheel" >
-    <mu1>0.3</mu1>
-    <mu2>0.3</mu2>
-    <kp>1000000.0</kp>
-    <kd>100.0</kd>
-    <minDepth>0.0</minDepth>
-    <maxContacts>1</maxContacts>
-  </gazebo>
-  <gazebo reference="right_front_wheel" >
-    <mu1>0.3</mu1>
-    <mu2>0.3</mu2>
-    <kp>1000000.0</kp>
-    <kd>100.0</kd>
-    <minDepth>0.0</minDepth>
-    <maxContacts>1</maxContacts>
-  </gazebo>
+<robot xmlns:xacro="http://wiki.ros.org/xacro" name="robot">
+    <xacro:include filename="$(find outdoor_robot_one)/description/inertial_macros.xacro"/>
+    <xacro:include filename="$(find outdoor_robot_one)/description/robot_gazebo.urdf.xacro"/>
+    <xacro:include filename="$(find outdoor_robot_one)/description/robot_core.urdf.xacro"/>
+    <xacro:include filename="$(find outdoor_robot_one)/description/robot_controller.ros2_control.xacro"/>
 </robot>

Commit message: added camera model to urdf

File: description/robot.urdf.xacro (robot description, xacro)
@@ -1,4 +1,6 @@
 <?xml version="1.0"?>
 <robot xmlns:xacro="http://wiki.ros.org/xacro" name="robot">
+    <xacro:arg name="use_nominal_extrinsics" default="false"/>
+    <xacro:include filename="$(find realsense2_description)/urdf/_d455.urdf.xacro" />
     <xacro:include filename="$(find outdoor_robot_one)/description/inertial_macros.xacro"/>
     <xacro:include filename="$(find outdoor_robot_one)/description/robot_gazebo.urdf.xacro"/>

File: description/robot_core.urdf.xacro (robot description, xacro)
@@ -120,3 +120,12 @@
   </xacro:inertial_cylinder>
   </link>
+  <joint name="camera_mount_joint" type="fixed">
+    <parent link="base_link" />
+    <child link="camera_mount_link" />
+    <origin xyz="0.32 0 0.18" />
+  </joint>
+  <link name="camera_mount_link" />
+  <xacro:sensor_d455 parent="camera_mount_link" use_nominal_extrinsics="$(arg use_nominal_extrinsics)">
+    <origin xyz="0 0 0" rpy="0 0 0"/>
+  </xacro:sensor_d455>
 </robot>
